File: hardware/analog_board/Power_Filter.kicad_sch (KiCad schematic)
At the start: 76 parts

Commit message: debug：修正原理图部分错误
Changed lines of the file:
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@@
 		(polyline
 			(pts
-				(xy 13.97 16.51) (xy 13.97 123.19) (xy 280.67 123.19) (xy 280.67 16.51)
+				(xy 13.97 16.51) (xy 13.97 123.19) (xy 280.67 121.92) (xy 280.67 16.51)
 			)
 			(stroke
@@
 		(in_pos_files yes)
 		(dnp no)
-		(fields_autoplaced yes)
 		(property "Reference" "#PWR0112"
 			(at 264.16 71.12 0)
@@
 		)
 		(property "Value" "Clock_V_{VCO}"
-			(at 266.7 66.0399 0)
+			(at 259.588 62.992 0)
 			(show_name no)
 			(do_not_autoplace no)
@@
 		(in_pos_files yes)
 		(dnp no)
-		(fields_autoplaced yes)
 		(property "Reference" "#PWR039"
 			(at 149.86 72.39 0)
@@
 		)
 		(property "Value" "+1.8VA_DAC"
-			(at 152.4 67.3099 0)
+			(at 144.018 64.008 0)
 			(show_name no)
 			(do_not_autoplace no)
@@
 		(in_pos_files yes)
 		(dnp no)
-		(fields_autoplaced yes)
 		(property "Reference" "#PWR045"
 			(at 149.86 99.06 0)
@@
 		)
 		(property "Value" "+1.8VD_DAC"
-			(at 152.4 93.9799 0)
+			(at 144.272 90.678 0)
 			(show_name no)
 			(do_not_autoplace no)
@@
 		(in_pos_files yes)
 		(dnp no)
-		(fields_autoplaced yes)
 		(property "Reference" "#PWR043"
 			(at 176.53 72.39 0)
@@
 		)
 		(property "Value" "+1.8VA_DAC"
-			(at 179.07 67.3099 0)
+			(at 171.196 64.008 0)
 			(show_name no)
 			(do_not_autoplace no)
@@
 		(in_pos_files yes)
 		(dnp no)
-		(fields_autoplaced yes)
 		(property "Reference" "#PWR0119"
 			(at 264.16 99.06 0)
@@
 		)
 		(property "Value" "Clock_V_{TCXO}"
-			(at 266.7 93.9799 0)
+			(at 259.334 90.678 0)
 			(show_name no)
 			(do_not_autoplace no)
@@
 		(in_pos_files yes)
 		(dnp no)
-		(fields_autoplaced yes)
 		(property "Reference" "#PWR047"
 			(at 25.4 97.79 0)
@@
 		)
 		(property "Value" "+3.3VA"
-			(at 27.94 92.7099 0)
+			(at 22.098 89.408 0)
 			(show_name no)
 			(do_not_autoplace no)
@@
 		(in_pos_files yes)
 		(dnp no)
-		(fields_autoplaced yes)
 		(property "Reference" "#PWR0107"
 			(at 227.33 71.12 0)
@@
 		)
 		(property "Value" "Clock_V_{DD}"
-			(at 229.87 66.0399 0)
+			(at 223.266 62.738 0)
 			(show_name no)
 			(do_not_autoplace no)
@@
 		(in_pos_files yes)
 		(dnp no)
-		(fields_autoplaced yes)
 		(property "Reference" "#PWR016"
 			(at 26.67 35.56 0)
@@
 		)
 		(property "Value" "+1V0"
-			(at 29.21 30.4799 0)
+			(at 23.876 27.686 0)
 			(show_name no)
 			(do_not_autoplace no)
@@
 		(in_pos_files yes)
 		(dnp no)
-		(fields_autoplaced yes)
 		(property "Reference" "#PWR048"
 			(at 176.53 99.06 0)
@@
 		)
 		(property "Value" "+1.8VD_DAC"
-			(at 179.07 93.9799 0)
+			(at 170.688 90.678 0)
 			(show_name no)
 			(do_not_autoplace no)
@@
 		(in_pos_files yes)
 		(dnp no)
-		(fields_autoplaced yes)
 		(property "Reference" "#PWR0116"
 			(at 227.33 99.06 0)
@@
 		)
 		(property "Value" "Clock_V_{DDIO}"
-			(at 229.87 93.9799 0)
+			(at 222.25 90.424 0)
 			(show_name no)
 			(do_not_autoplace no)
@@
 		(in_pos_files yes)
 		(dnp no)
-		(fields_autoplaced yes)
 		(property "Reference" "#PWR027"
 			(at 187.96 35.56 0)
@@
 		)
 		(property "Value" "+3.3V"
-			(at 190.5 30.4799 0)
+			(at 185.166 27.432 0)
 			(show_name no)
 			(do_not_autoplace no)
@@
 		(in_pos_files yes)
 		(dnp no)
-		(fields_autoplaced yes)
 		(property "Reference" "#PWR050"
 			(at 125.73 97.79 0)
@@
 		)
 		(property "Value" "+1.8VD"
-			(at 128.27 92.7099 0)
+			(at 122.174 89.154 0)
 			(show_name no)
 			(do_not_autoplace no)
@@
 		(in_pos_files yes)
 		(dnp no)
-		(fields_autoplaced yes)
 		(property "Reference" "#PWR041"
 			(at 125.73 71.12 0)
@@
 		)
 		(property "Value" "+1.8VA"
-			(at 128.27 66.0399 0)
+			(at 121.92 62.23 0)
 			(show_name no)
 			(do_not_autoplace no)
@@
 		(in_pos_files yes)
 		(dnp no)
-		(fields_autoplaced yes)
 		(property "Reference" "#PWR023"
 			(at 124.46 35.56 0)
@@
 		)
 		(property "Value" "+1V0"
-			(at 127 30.4799 0)
+			(at 121.92 27.432 0)
 			(show_name no)
 			(do_not_autoplace no)
@@
 		(in_pos_files yes)
 		(dnp no)
-		(fields_autoplaced yes)
 		(property "Reference" "#PWR017"
 			(at 81.28 35.56 0)
@@
 		)
 		(property "Value" "+1V0"
-			(at 83.82 30.4799 0)
+			(at 78.232 27.686 0)
 			(show_name no)
 			(do_not_autoplace no)
