File: hardware/analog_board/analog_board.kicad_sch (KiCad schematic)
At the start: 6 parts, among them J2 Conn_02x08_Counter_Clockwise, J4 Conn_01x08, J5 CH1, J6 CH1

Commit message: feat：BOM导出
Parts:
- J5, J6: value CH1 -> SMA
Changed lines of the file:
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@@
 			)
 		)
-		(property "Value" "CH1"
+		(property "Value" "SMA"
 			(at 159.766 78.74 0)
 			(show_name no)
@@
 			)
 		)
-		(property "Value" "CH1"
+		(property "Value" "SMA"
 			(at 159.766 83.82 0)
 			(show_name no)
