File: hardware/control_board/control_board/control_board.kicad_sch (KiCad schematic)
At the start: 6 parts, among them J1 USB_B, J2 Conn_02x08_Counter_Clockwise, J5 Conn_01x08

Commit message: debug：修复原理图部分问题
Parts:
- added H1, H2, H3, H4: M3, MountingHole:MountingHole_3.2mm_M3, symbol Mechanical:MountingHole
