File: hardware/control_board/control_board/control_board.kicad_pcb (KiCad board)
At the start: 4 copper layers, 100 x 100 mm, 144 parts, among them J1 USB_B, J2 Conn_02x08_Counter_Clockwise, J3 Conn_01x06_Pin, J4 Barrel_Jack_Switch, J5 Conn_01x08, Q1 SS8550, Q2 AO3401A, SW1 BOOT0, SW2 NRST, U1 STM32F411CEUx, U2 M24C64, U3 TPS54360DDA, U4 TPS54360DDA, U5 TPS54360DDA, U6 TPS54360DDA, U7 TPS62933, Y1 25MHz, Y2 32.768kHz

Commit message: debug：修改 PCB 部分问题
Parts:
- added H1: M3, MountingHole:MountingHole_3.2mm_M3, F.Cu at (25.0, 25.0)
- added H2: M3, MountingHole:MountingHole_3.2mm_M3, F.Cu at (115.0, 25.0)
- added H3: M3, MountingHole:MountingHole_3.2mm_M3, F.Cu at (25.0, 105.0)
- added H4: M3, MountingHole:MountingHole_3.2mm_M3, F.Cu at (100.0, 60.0)
- added J6: Conn_01x02_Pin, Connector_JST:JST_VH_B2P-VH-B_1x02_P3.96mm_Vertical, F.Cu at (41.3, 60.3)
- BT1: footprint Battery:BatteryHolder_Keystone_1060_1x2032 -> ArbWave30:BAT-TH_BS-05-A1BJ001
- C15, C24, C37, C47: value 22uF -> 35V 22uF
- C3, C4: value 30p -> 10p
- D5, D6, D7, D8: value SS34 -> SS36
- R13: value 77.5k -> 75k
- R21: value 77.5kR -> 75kR
- Y2: footprint Crystal:Crystal_SMD_3225-4Pin_3.2x2.5mm -> Crystal:Crystal_SMD_3215-2Pin_3.2x1.5mm
- moved BT1 58.9 mm to (44.7, 26.5)
- moved Q2 31.5 mm to (59.9, 29.4), turned to 90 degrees
- moved R4 30.3 mm to (56.0, 32.6), turned to 0 degrees
- moved D3 25.7 mm to (59.9, 32.6), turned to 180 degrees
- moved J3 20.6 mm to (50.0, 43.2), turned to 90 degrees
- moved BZ1 18.0 mm to (74.3, 28.1)
- moved Q1 18.0 mm to (79.7, 28.1)
- moved D9 18.0 mm to (80.4, 24.8)
- moved R30 18.0 mm to (84.0, 28.1)
- moved R31 18.0 mm to (82.4, 28.1)
- moved D4 17.6 mm to (46.1, 58.2), turned to 90 degrees
- moved C61 17.5 mm to (63.4, 62.1)
- moved C64 17.5 mm to (68.7, 59.3)
- moved R29 17.5 mm to (58.9, 56.0)
- moved C60 17.5 mm to (62.8, 53.0)
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Connections:
- J4 pad 1: V_{IN} -> Net-(J6-Pin_2)
- Y2 pad 2: GND -> /MCU/OSC32_OUT
Routing:
- net /MCU/Debug_RX: track 31.2 -> 46.3 mm
- net /MCU/Buzzer: track 28.8 -> 14.4 mm
- net /MCU/Debug_TX: track 29.8 -> 42.2 mm
- net /MCU/Debug_LED: track 22.4 -> 11.0 mm
- net /MCU/SWCLK: track 29.1 -> 39.6 mm
- net /FPGA_Ctrl.Ctrl_SPI_CLK: track 20.7 -> 25.8 mm
- net /FPGA_Ctrl.Ctrl_SPI_CS: track 24.7 -> 29.7 mm
- net /FPGA_Ctrl.Ctrl_SPI_MISO: track 24.5 -> 29.5 mm
- net /FPGA_Ctrl.Ctrl_FPGA_NRST: track 22.5 -> 26.9 mm
- net /MCU/NRST: track 79.3 -> 83.4 mm
- net /FPGA_Ctrl.Ctrl_SPI_MOSI: track 19.9 -> 23.9 mm
- net /FPGA_Ctrl.GPIO1: track 22.2 -> 26.1 mm
- net /FPGA_Ctrl.GPIO2: track 21.9 -> 25.8 mm
- net /MCU/SWDIO: track 29.7 -> 32.1 mm
- net /MCU/OSC32_OUT: track 9.18 -> 7.34 mm
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- added copper zone on F.Cu, net Net-(J6-Pin_2)
Other:
- board size 100 x 100 mm -> 100 x 90 mm
