File: hardware/control_board/control_board/POWER.kicad_sch (KiCad schematic)
At the start: 94 parts, among them J4 Barrel_Jack_Switch, U3 TPS54360DDA, U4 TPS54360DDA, U5 TPS54360DDA, U6 TPS54360DDA, U7 TPS62933

Commit message: debug：修复原理图部分问题
Parts:
- removed D5, D6, D7, D8: SS34, Diode_SMD:D_SMA, symbol Diode:SS34
- added D5, D6, D7, D8: SS36, Diode_SMD:D_SMA, symbol Diode:SS36
- added J6: Conn_01x02_Pin, Connector_JST:JST_VH_B2P-VH-B_1x02_P3.96mm_Vertical, symbol Connector:Conn_01x02_Pin
- C15, C24, C37, C47: value 22uF -> 35V 22uF
- R13: value 77.5k -> 75k
- R21: value 77.5kR -> 75kR
Connections:
- net -17V: now also D8.2 (A)
- net -7V: now also D7.2 (A)
- net GND: now also D5.2 (A), D6.2 (A)
- net V_{IN}: now also J6.1 (Pin_1); no longer J4.1
- net at C36.1, L3.1, U5.8 (SW): now also D7.1 (K)
- net at C46.1, L4.1, U6.8 (SW): now also D8.1 (K)
- net at C14.1, L1.1, U3.8 (SW): now also D5.1 (K)
- net at C23.1, L2.1, U4.8 (SW): now also D6.1 (K)
- new net: J4.1, J6.2 (Pin_2)
Other:
- moved on the sheet: C15, C24, C37, C46, C47, C48, C49, C50, C51, C52, C53, C54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

Commit message: feat：给出BOM表
Parts:
- TP10, TP11, TP7, TP8, TP9: now left out of the parts list
Changed lines of the file:
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@@
 		(body_style 1)
 		(exclude_from_sim no)
-		(in_bom yes)
+		(in_bom no)
 		(on_board yes)
 		(in_pos_files yes)
@@
 		(body_style 1)
 		(exclude_from_sim no)
-		(in_bom yes)
+		(in_bom no)
 		(on_board yes)
 		(in_pos_files yes)
@@
 		(body_style 1)
 		(exclude_from_sim no)
-		(in_bom yes)
+		(in_bom no)
 		(on_board yes)
 		(in_pos_files yes)
@@
 		(body_style 1)
 		(exclude_from_sim no)
-		(in_bom yes)
+		(in_bom no)
 		(on_board yes)
 		(in_pos_files yes)
@@
 		(body_style 1)
 		(exclude_from_sim no)
-		(in_bom yes)
+		(in_bom no)
 		(on_board yes)
 		(in_pos_files yes)
